File: Cherry-Mx-Bitboard-Re-19.05mm/Cherry-Mx-Bitboard-Re-19.05mm.sch (KiCad schematic (older format))
At the start: 11 parts, among them SW1 SW_Push

Commit message: remove unused kicad projects
Parts:
- D2: footprint Diode_SMD:D_SOD-323_HandSoldering -> Footprints:1N4148W
Changed lines of the file:
@@
 F 0 "D2" H 2400 4683 50  0000 C CNN
 F 1 "1N4148W" H 2400 4774 50  0000 C CNN
-F 2 "Diode_SMD:D_SOD-323_HandSoldering" H 2400 4725 50  0001 C CNN
+F 2 "Footprints:1N4148W" H 2400 4725 50  0001 C CNN
 F 3 "https://www.vishay.com/docs/85748/1n4148w.pdf" H 2400 4900 50  0001 C CNN
 	1    2400 4900
